File: Sweep High M/sweep-high.kicad_pcb (KiCad board)
At the start: 2 copper layers, 113.5 x 95.2 mm, 25 parts, among them J2 AudioJack4dpb, SW10 SW_Push, SW11 SW_Push, SW12 SW_Push, SW14 SW_Push, SW15 SW_Push, SW16 SW_Push, SW17 SW_Push, SW18 SW_Push, SW2 SW_Push, SW2 SW_SPDT, SW20 SW_Push, SW21 SW_Push, SW3 SW_Push, SW4 SW_Push, SW5 SW_Push, SW6 SW_Push, SW8 SW_Push, SW9 SW_Push, U1 ProMicro-kbd

Commit message: kicad 7 and rounded tracks for M
Parts:
- moved U1 1.00 mm to (141.1, 100.2)
Routing:
- net Switch6: track 127.5 -> 158.8 mm
- net Switch2: track 98.0 -> 124.7 mm
- net Switch11: track 149.3 -> 169.7 mm
- net Switch15: track 48.0 -> 67.6 mm
- net Switch3: track 82.8 -> 101.2 mm
- net Switch8: track 81.8 -> 99.4 mm
- net Switch4: track 60.0 -> 76.6 mm
- net Switch1: track 175.0 -> 190.5 mm
- net Switch7: track 107.5 -> 122.9 mm
- net Switch12: track 122.9 -> 138.0 mm
- net Switch14: track 77.3 -> 91.7 mm
- net reset: track 50.6 -> 64.4 mm
- net Switch5: track 48.2 -> 60.8 mm
- net Switch13: track 100.3 -> 110.8 mm
- net Switch16: track 53.4 -> 59.1 mm
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Other:
- board size 113.5 x 95.2 mm -> 114.5 x 95.3 mm
