File: Sweep High M/sweep-high.kicad_pcb (KiCad board)
At the start: 2 copper layers, 114.5 x 95.3 mm, 25 parts, among them J2 AudioJack4dpb, SW10 SW_Push, SW11 SW_Push, SW12 SW_Push, SW14 SW_Push, SW15 SW_Push, SW16 SW_Push, SW17 SW_Push, SW18 SW_Push, SW2 SW_Push, SW2 SW_SPDT, SW20 SW_Push, SW21 SW_Push, SW3 SW_Push, SW4 SW_Push, SW5 SW_Push, SW6 SW_Push, SW8 SW_Push, SW9 SW_Push, U1 ProMicro-kbd

Commit message: update
Changed lines of the file:
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@@
   (segment (start 110.74 116.54) (end 110.133349 117.146651) (width 0.25) (layer "F.Cu") (net 20))
   (segment (start 146.48 111.74) (end 146.48 121.82) (width 0.25) (layer "F.Cu") (net 20))
-  (segment (start 141.54 124.42) (end 142.635 123.325) (width 0.25) (layer "F.Cu") (net 21))
+  (segment (start 131.290295 124.369705) (end 131.290295 126.834591) (width 0.25) (layer "F.Cu") (net 21))
   (segment (start 129.355409 126.834591) (end 128.920443 127.269557) (width 0.25) (layer "F.Cu") (net 21))
-  (segment (start 147.01 114.23) (end 147.532 113.708) (width 0.25) (layer "F.Cu") (net 21))
-  (segment (start 131.290295 126.834591) (end 140.805409 126.834591) (width 0.25) (layer "F.Cu") (net 21))
-  (segment (start 140.805409 126.834591) (end 141.54 126.1) (width 0.25) (layer "F.Cu") (net 21))
+  (segment (start 147.01 122.55) (end 146.235 123.325) (width 0.25) (layer "F.Cu") (net 21))
   (segment (start 128.920443 127.269557) (end 128.920443 128.399295) (width 0.25) (layer "F.Cu") (net 21))
   (segment (start 131.290295 126.834591) (end 129.355409 126.834591) (width 0.25) (layer "F.Cu") (net 21))
-  (segment (start 146.235 123.325) (end 147.01 122.55) (width 0.25) (layer "F.Cu") (net 21))
-  (segment (start 147.01 122.55) (end 147.01 114.23) (width 0.25) (layer "F.Cu") (net 21))
-  (segment (start 147.532 113.708) (end 148.7054 113.708) (width 0.25) (layer "F.Cu") (net 21))
-  (segment (start 141.54 126.1) (end 141.54 124.42) (width 0.25) (layer "F.Cu") (net 21))
-  (segment (start 142.635 123.325) (end 146.235 123.325) (width 0.25) (layer "F.Cu") (net 21))
+  (segment (start 148.7054 113.708) (end 147.532 113.708) (width 0.25) (layer "F.Cu") (net 21))
+  (segment (start 147.532 113.708) (end 147.01 114.23) (width 0.25) (layer "F.Cu") (net 21))
+  (segment (start 146.235 123.325) (end 132.335 123.325) (width 0.25) (layer "F.Cu") (net 21))
+  (segment (start 132.335 123.325) (end 131.290295 124.369705) (width 0.25) (layer "F.Cu") (net 21))
+  (segment (start 147.01 114.23) (end 147.01 122.55) (width 0.25) (layer "F.Cu") (net 21))
   (segment (start 133.7824 86.065) (end 138.352 86.065) (width 0.25) (layer "F.Cu") (net 22))
   (segment (start 142.852 87.118) (end 142.852 86.065) (width 0.25) (layer "B.Cu") (net 22))
